File: hardware/LoRaPagerESP32.kicad_pcb (KiCad board)
At the start: 2 copper layers, 69 x 94.6 mm, 75 parts, among them J1 USB_C_Receptacle_USB2.0, J2 Conn_01x02, J3 Conn_01x03, J4 Conn_01x20_Male, J5 Conn_01x02, J6 Conn_01x02, J7 Conn_Coaxial, Q1 BSS84, Q2 BSS138, Q3 Q_NPN_BEC, Q4 Q_NPN_BEC, Q5 Q_NMOS_GSD, Q6 Q_PMOS_GSD, Q7 Q_PMOS_GSD, Q8 Q_NMOS_GSD, SW1 5W_SW, SW2 SW_Push, U1 PCA9555PW,118, U2 MCP73831-2-OT, U3 AP2112K-3.3, U4 ESP-32_WROOM32, U5 RFM96, U6 CP2104

Commit message: Version 1.1
Parts:
- removed C21: 1uF, Capacitor_SMD:C_0603_1608Metric
- removed J6: Conn_01x02, Connector_PinHeader_2.54mm:PinHeader_1x02_P2.54mm_Vertical
- added C26: 0.1uF, Capacitor_SMD:C_0603_1608Metric, B.Cu at (92.2, 39.3)
- added C27: 0.1uF, Capacitor_SMD:C_0603_1608Metric, B.Cu at (106.6, 69.1)
- added D4: LED, LED_SMD:LED_0603_1608Metric, B.Cu at (117.4, 70.7)
- added D5: LED, LED_SMD:LED_0603_1608Metric, B.Cu at (111.6, 70.7)
- added D6: LED, LED_SMD:LED_0603_1608Metric, B.Cu at (114.5, 70.7)
- added JP3: Jumper_NC_Small, modules:Test_bridge_2.54mm, F.Cu at (116.7, 113.3)
- added R17: 4.7k, Resistor_SMD:R_0603_1608Metric, B.Cu at (89.2, 65.1)
- added R18: 4.7k, Resistor_SMD:R_0603_1608Metric, B.Cu at (90.9, 65.1)
- added R19: 10k, Resistor_SMD:R_0603_1608Metric, B.Cu at (108.5, 67.3)
- added R20: 10k, Resistor_SMD:R_0603_1608Metric, B.Cu at (96.4, 66.5)
- added R21: 1k, Resistor_SMD:R_0603_1608Metric, B.Cu at (117.4, 75.1)
- added R22: 1k, Resistor_SMD:R_0603_1608Metric, B.Cu at (111.6, 75.1)
- added R23: 1k, Resistor_SMD:R_0603_1608Metric, B.Cu at (114.5, 75.1)
- added R24: 47.5k, Resistor_SMD:R_0603_1608Metric, B.Cu at (61.0, 63.0)
- added R25: 22.1k, Resistor_SMD:R_0603_1608Metric, B.Cu at (61.0, 64.6)
- added SW3: SW_Push, modules:1TS009, F.Cu at (113.1, 78.8)
- D1: footprint Diode_SMD:D_SOD-323 -> Diode_SMD:D_SOD-123
- R1: value 5K -> 5k
- R2, R3, R4, R5, R6: value 10K -> 10k
- moved R9 8.07 mm to (61.5, 71.0), turned to 180 degrees
- moved J2 6.79 mm to (105.6, 78.0), turned to 180 degrees
- moved C22 6.21 mm to (67.2, 59.9), turned to 0 degrees
- moved Q3 3.71 mm to (103.9, 69.1), turned to 180 degrees
- moved AE1 2.50 mm to (52.5, 30.0)
- moved Q4 2.08 mm to (99.2, 69.1)
- moved R5 2.06 mm to (101.5, 71.8)
- moved JP1 1.89 mm to (73.4, 56.0)
- moved C6 1.78 mm to (64.7, 69.8), turned to 270 degrees
- moved C4 1.33 mm to (61.0, 66.3)
- moved C5 1.31 mm to (61.0, 67.9)
- moved SW2 0.90 mm to (117.0, 36.3)
- moved C8 0.80 mm to (90.1, 67.4)
- moved D1 0.67 mm to (105.4, 116.6)
- moved C10 0.60 mm to (90.7, 69.9)
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Connections:
- C6 pad 1: Net-(C6-Pad1) -> VDD
- J2 pad 1: +BATT -> Net-(J2-Pad1)
- J3 pad 1: +BATT -> Net-(J2-Pad1)
- J5 pad 1: +3V3 -> /Display/LEDK
- J5 pad 2: /Display/LEDK -> +3V3
- R9 pad 1: VBUS -> VDD
- U1 pad 18: Net-(U1-Pad18) -> /Keyboard/KB_COL6
- U4 pad 6: /KB_LED -> Net-(U4-Pad6)
- U4 pad 8: Net-(U4-Pad8) -> /KB_LED
- U4 pad 9: Net-(U4-Pad9) -> /HEARTBEAT_LED
- U6 pad 5: Net-(C6-Pad1) -> VDD
- U6 pad 6: Net-(C6-Pad1) -> VDD
- U6 pad 8: VBUS -> Net-(R24-Pad1)
Routing:
- net Net-(J2-Pad1): track 0.00 -> 41.7 mm
- net +BATT: track 69.9 -> 29.7 mm
- net /Keyboard/KB_COL6: track 0.00 -> 39.6 mm, vias 0 -> 1
- net /HEARTBEAT_LED: track 0.00 -> 20.8 mm, vias 0 -> 2
- net GND: track 62.9 -> 46.3 mm, vias 67 -> 75
- net Net-(R9-Pad2): track 7.59 -> 17.8 mm
- net /RFM_INT: track 83.3 -> 74.2 mm, vias 1 -> 3
- net VBUS: track 132.6 -> 124.6 mm
- net /Power/EN: track 107.6 -> 115.1 mm
- net VDD: track 0.00 -> 7.33 mm
- net /RESET: track 13.7 -> 20.8 mm
- net /Keyboard/KB_ROW8: track 61.5 -> 67.8 mm
- net /Power/VIN: track 111.6 -> 116.4 mm
- net /GPIO0: track 32.7 -> 36.9 mm
- net Net-(R24-Pad1): track 0.00 -> 3.94 mm
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Other:
- outline, holes or cut-outs redrawn
- board text added: "LoRa ESP32 experimenter board Victor Joukov github.com/victzh Jan 2019 v1.1"
- board text removed: "LoRa ESP32 experimeter board v1 Victor Joukov github.com/victzh Dec 2018"
